Commit message: Initial rgbd camera implementation

File: models/hippo3/urdf/hippo3.xacro (robot description, xacro)
@@ -7,4 +7,5 @@
     <xacro:include filename="$(find hippo_sim)/models/hippo3/urdf/mount_macro.xacro" />
     <xacro:include filename="$(find hippo_sim)/models/camera/urdf/camera_macro.xacro" />
+    <xacro:include filename="$(find hippo_sim)/models/camera/urdf/rgbd_camera_macro.xacro" />
     <xacro:include filename="$(find hippo_sim)/models/acoustic_modem/urdf/acoustic_modem_macro.xacro" />
     <xacro:property name="thruster_xy" value="${thruster_r / 2**0.5}" />
@@ -115,4 +116,10 @@
             xyz="${vertical_camera_position}" rpy="${vertical_camera_orientation}" />
     </xacro:if>
+    <xacro:if value="$(arg use_rgbd_camera)">
+        <xacro:rgbd_camera_macro parent="base_link"
+            prefix="rgbd_camera" topic_prefix="$(arg vehicle_name)/rgbd_camera"
+            ignition_frame_id="$(arg vehicle_name)::rgbd_camera"
+            xyz="${rgbd_camera_position}" rpy="${rgbd_camera_orientation}" />
+    </xacro:if>
     <xacro:if value="$(arg use_acoustic_modem)">
         <xacro:acoustic_modem_macro parent="base_link"

File: models/hippo3/urdf/hippo3_params.xacro (robot description, xacro)
@@ -13,4 +13,7 @@
     <xacro:property name="vertical_camera_position" value="0.15 0.0 -0.03" />
     <xacro:property name="vertical_camera_orientation" value="0 ${radians(90)} 0" />
+    <xacro:arg name="use_rgbd_camera" default="false" />
+    <xacro:property name="rgbd_camera_position" value="0.2 0.0 0.0" />
+    <xacro:property name="rgbd_camera_orientation" value="0 0 0" />
     <xacro:arg name="use_acoustic_modem" default="false" />
     <xacro:property name="modem_position" value="0 0 -0.1" />
